Commit message: Fix urdf

File: urdf/robot.urdf (robot description, URDF)
Before this commit: robot robot, 52 links, 51 joints
Links:
- link link_Head: geometry collision mesh filename=c_Head.stl scale=1.0 1.0 1.0; visual mesh filename=Head.stl scale=1.0 1.0 1.0
- link link_Hips: geometry collision mesh filename=c_Hips.stl scale=1.0 1.0 1.0; visual mesh filename=Hips.stl scale=1.0 1.0 1.0
- link link_LeftArm: geometry collision mesh filename=c_LeftArm.stl scale=1.0 1.0 1.0; visual mesh filename=LeftArm.stl scale=1.0 1.0 1.0
- link link_LeftFoot: geometry collision mesh filename=c_LeftFoot.stl scale=1.0 1.0 1.0; visual mesh filename=LeftFoot.stl scale=1.0 1.0 1.0
- link link_LeftForeArm: geometry collision mesh filename=c_LeftForeArm.stl scale=1.0 1.0 1.0; visual mesh filename=LeftForeArm.stl scale=1.0 1.0 1.0
- link link_LeftHand: geometry collision mesh filename=c_LeftHand.stl scale=1.0 1.0 1.0; visual mesh filename=LeftHand.stl scale=1.0 1.0 1.0
- link link_LeftHandIndex1: geometry collision mesh filename=c_LeftHandIndex.stl scale=1.0 1.0 1.0; visual mesh filename=LeftHandIndex1.stl scale=1.0 1.0 1.0
- link link_LeftHandIndex2: geometry collision mesh filename=c_LeftHandIndex2.stl scale=1.0 1.0 1.0; visual mesh filename=LeftHandIndex2.stl scale=1.0 1.0 1.0
- link link_LeftHandIndex3: geometry collision mesh filename=c_LeftHandIndex3.stl scale=1.0 1.0 1.0; visual mesh filename=LeftHandIndex3.stl scale=1.0 1.0 1.0
- link link_LeftHandMiddle1: geometry collision mesh filename=c_LeftHandMiddle1.stl scale=1.0 1.0 1.0; visual mesh filename=LeftHandMiddle1.stl scale=1.0 1.0 1.0
- link link_LeftHandMiddle2: geometry collision mesh filename=c_LeftHandMiddle2.stl scale=1.0 1.0 1.0; visual mesh filename=LeftHandMiddle2.stl scale=1.0 1.0 1.0
- link link_LeftHandMiddle3: geometry collision mesh filename=c_LeftHandMiddle3.stl scale=1.0 1.0 1.0; visual mesh filename=LeftHandMiddle3.stl scale=1.0 1.0 1.0
- link link_LeftHandPinky1: geometry collision mesh filename=c_LeftHandPinky1.stl scale=1.0 1.0 1.0; visual mesh filename=LeftHandPinky1.stl scale=1.0 1.0 1.0
- link link_LeftHandPinky2: geometry collision mesh filename=c_LeftHandPinky2.stl scale=1.0 1.0 1.0; visual mesh filename=LeftHandPinky2.stl scale=1.0 1.0 1.0
- link link_LeftHandPinky3: geometry collision mesh filename=c_LeftHandPinky3.stl scale=1.0 1.0 1.0; visual mesh filename=LeftHandPinky3.stl scale=1.0 1.0 1.0
- link link_LeftHandRing1: geometry collision mesh filename=c_LeftHandRing1.stl scale=1.0 1.0 1.0; visual mesh filename=LeftHandRing1.stl scale=1.0 1.0 1.0
- link link_LeftHandRing2: geometry collision mesh filename=c_LeftHandRing2.stl scale=1.0 1.0 1.0; visual mesh filename=LeftHandRing2.stl scale=1.0 1.0 1.0
- link link_LeftHandRing3: geometry collision mesh filename=c_LeftHandRing3.stl scale=1.0 1.0 1.0; visual mesh filename=LeftHandRing3.stl scale=1.0 1.0 1.0
- link link_LeftHandThumb1: geometry collision mesh filename=c_LeftHandThumb1.001.stl scale=1.0 1.0 1.0; collision sphere radius=0.01773
- link link_LeftHandThumb2: geometry collision mesh filename=c_LeftHandThumb2.001.stl scale=0.01 0.01 0.01; collision sphere radius=0.01069
- link link_LeftHandThumb3: geometry collision mesh filename=c_LeftHandThumb3.001.stl scale=1.0 1.0 1.0; collision sphere radius=0.00798
- link link_LeftLeg: geometry collision mesh filename=c_LeftLeg.stl scale=1.0 1.0 1.0; visual mesh filename=LeftLeg.stl scale=1.0 1.0 1.0
- link link_LeftShoulder: geometry collision sphere radius=0.04861; visual mesh filename=LeftShoulder.stl scale=1.0 1.0 1.0
- link link_LeftToeBase: geometry collision mesh filename=c_LeftToeBase.stl scale=1.0 1.0 1.0; visual mesh filename=LeftToeBase.stl scale=1.0 1.0 1.0
- link link_LeftUpLeg: geometry collision mesh filename=c_LeftUpLeg.stl scale=1.0 1.0 1.0; visual mesh filename=LeftUpLeg.stl scale=1.0 1.0 1.0
- link link_Neck: geometry collision sphere radius=0.05128; visual mesh filename=Neck.stl scale=1.0 1.0 1.0
- link link_RightArm: geometry collision mesh filename=c_RightArm.stl scale=1.0 1.0 1.0; visual mesh filename=RightArm.stl scale=1.0 1.0 1.0
- link link_RightFoot: geometry collision mesh filename=c_RightFoot.stl scale=1.0 1.0 1.0; visual mesh filename=RightFoot.stl scale=1.0 1.0 1.0
- link link_RightForeArm: geometry collision mesh filename=c_RightForeArm.stl scale=1.0 1.0 1.0; visual mesh filename=RightForeArm.stl scale=1.0 1.0 1.0
- link link_RightHand: geometry collision mesh filename=c_RightHand.stl scale=1.0 1.0 1.0; visual mesh filename=RightHand.stl scale=1.0 1.0 1.0
- link link_RightHandIndex1: geometry collision mesh filename=c_RightHandIndex1.stl scale=1.0 1.0 1.0; visual mesh filename=RightHandIndex1.stl scale=1.0 1.0 1.0
- link link_RightHandIndex2: geometry collision mesh filename=c_RightHandIndex2.stl scale=1.0 1.0 1.0; visual mesh filename=RightHandIndex2.stl scale=1.0 1.0 1.0
- link link_RightHandIndex3: geometry collision mesh filename=c_RightHandIndex3.stl scale=1.0 1.0 1.0; visual mesh filename=RightHandIndex3.stl scale=1.0 1.0 1.0
- link link_RightHandMiddle1: geometry collision mesh filename=c_RightHandMiddle1.stl scale=1.0 1.0 1.0; visual mesh filename=RightHandMiddle1.stl scale=1.0 1.0 1.0
- link link_RightHandMiddle2: geometry collision mesh filename=c_RightHandMiddle2.stl scale=1.0 1.0 1.0; visual mesh filename=RightHandMiddle2.stl scale=1.0 1.0 1.0
- link link_RightHandMiddle3: geometry collision mesh filename=c_RightHandMiddle3.stl scale=1.0 1.0 1.0; visual mesh filename=RightHandMiddle3.stl scale=1.0 1.0 1.0
- link link_RightHandPinky1: geometry collision mesh filename=c_RightHandPinky1.stl scale=1.0 1.0 1.0; visual mesh filename=RightHandPinky1.stl scale=1.0 1.0 1.0
- link link_RightHandPinky2: geometry collision mesh filename=c_RightHandPinky2.stl scale=1.0 1.0 1.0; visual mesh filename=RightHandPinky2.stl scale=1.0 1.0 1.0
- link link_RightHandPinky3: geometry collision mesh filename=c_RightHandPinky3.stl scale=1.0 1.0 1.0; visual mesh filename=RightHandPinky3.stl scale=1.0 1.0 1.0
- link link_RightHandRing1: geometry collision mesh filename=c_RightHandRing1.stl scale=1.0 1.0 1.0; visual mesh filename=RightHandRing1.stl scale=1.0 1.0 1.0
- link link_RightHandRing2: geometry collision mesh filename=c_RightHandRing2.stl scale=1.0 1.0 1.0; visual mesh filename=RightHandRing2.stl scale=1.0 1.0 1.0
- link link_RightHandRing3: geometry collision mesh filename=c_RightHandRing3.stl scale=1.0 1.0 1.0; visual mesh filename=RightHandRing3.stl scale=1.0 1.0 1.0
- link link_RightHandThumb1: geometry collision mesh filename=c_RightHandThumb1.stl scale=1.0 1.0 1.0; visual mesh filename=RightHandThumb1.stl scale=1.0 1.0 1.0
- link link_RightHandThumb2: geometry collision mesh filename=c_RightHandThumb2.001.stl scale=1.0 1.0 1.0; collision sphere radius=0.01094
- link link_RightHandThumb3: geometry collision mesh filename=c_RightHandThumb3.001.stl scale=1.0 1.0 1.0; collision sphere radius=0.00816
- link link_RightLeg: geometry collision mesh filename=c_RightLeg.stl scale=1.0 1.0 1.0; visual mesh filename=RightLeg.stl scale=1.0 1.0 1.0
- link link_RightShoulder: geometry collision sphere radius=0.04861; visual mesh filename=RightShoulder.stl scale=1.0 1.0 1.0
- link link_RightToeBase: geometry collision mesh filename=c_RightToeBase.stl scale=1.0 1.0 1.0; visual mesh filename=RightToeBase.stl scale=1.0 1.0 1.0
- link link_RightUpLeg: geometry collision mesh filename=c_RightUpLeg.stl scale=1.0 1.0 1.0; visual mesh filename=RightUpLeg.stl scale=1.0 1.0 1.0
- link link_Spine: geometry collision mesh filename=c_Spine.stl scale=1.0 1.0 1.0; visual mesh filename=Spine.stl scale=1.0 1.0 1.0
- link link_Spine1: geometry collision sphere radius=0.10869; visual mesh filename=Spine1.stl scale=1.0 1.0 1.0
- link link_Spine2: geometry collision mesh filename=c_Spine2.stl scale=1.0 1.0 1.0; visual mesh filename=Spine2.stl scale=1.0 1.0 1.0
Joints:
- joint link_Head: origin xyz=0 0 0 rpy=0 0 0 -> xyz=0 0 0 rpy=1.5708 0 0
- joint link_LeftUpLeg: origin xyz=0 0 0 rpy=0 0 0 -> xyz=0 0.02076 -1.09271 rpy=0 0 0
- joint link_Neck: limit (none) -> effort=200.0 velocity=40.0; type fixed -> floating
- joint link_RightLeg: origin xyz=0 0 0 rpy=0 0 0 -> xyz=0.08208 0.00477 -1.19426 rpy=0 0 0
- joint link_RightUpLeg: origin xyz=0 0 0 rpy=0 0 0 -> xyz=-0.08208 0.016 0.10154 rpy=0 0 0
- joint link_Spine: origin xyz=0 0 0 rpy=0 0 0 -> xyz=0 -0.00132 0.09968 rpy=0 0 0
- joint link_Spine1: limit (none) -> effort=500.0 velocity=40.0; origin xyz=0 0 0 rpy=0 0 0 -> xyz=0 0.01001 0.09618 rpy=0 0 0; type fixed -> floating
- joint link_Spine2: limit (none) -> effort=200.0 velocity=40.0; origin xyz=0 0 0 rpy=0 0 0 -> xyz=0 0.01207 -1.28858 rpy=0 0 0; type fixed -> floating

Commit message: Update robot.urdf, add example

File: urdf/robot.urdf (robot description, URDF)
Before this commit: robot robot, 52 links, 51 joints
Joints:
- joint link_Head: origin xyz=0 0 0 rpy=1.5708 0 0 -> xyz=0 0 1.6 rpy=1.5708 0 0
- joint link_LeftArm: origin xyz=0 0 0 rpy=0 0 0 -> xyz=0.1519 0.0513 1.4367 rpy=0 0 0; type fixed -> spherical
- joint link_LeftFoot: origin xyz=0 0 0 rpy=0 0 0 -> xyz=0.083248 0.021837 0.083976 rpy=0 0 0; type fixed -> spherical
- joint link_LeftForeArm: axis (none) -> 0.000000 0.000000 1.000000; limit (none) -> lower=0 upper=3.14 effort=1000.0 velocity=0.5; origin xyz=0 0 0 rpy=0 0 0 -> xyz=0.4308 0.0513 1.4377 rpy=0 0 0; type fixed -> revolute
- joint link_LeftHand: origin xyz=0 0 0 rpy=0 0 0 -> xyz=0.713253 0.050178 1.43734 rpy=0 0 0; type fixed -> spherical
- joint link_LeftHandIndex1: origin xyz=0 0 0 rpy=0 0 0 -> xyz=0.804532 0.026772 1.43359 rpy=0 0 0
- joint link_LeftHandIndex2: origin xyz=0 0 0 rpy=0 0 0 -> xyz=0.841082 0.027373 1.43234 rpy=0 0 0
- joint link_LeftHandIndex3: origin xyz=0 0 0 rpy=0 0 0 -> xyz=0.869889 0.027973 1.43275 rpy=0 0 0
- joint link_LeftHandMiddle1: origin xyz=0 0 0 rpy=0 0 0 -> xyz=0.808261 0.050178 1.43796 rpy=0 0 0
- joint link_LeftHandMiddle2: origin xyz=0 0 0 rpy=0 0 0 -> xyz=0.845307 0.050178 1.43738 rpy=0 0 0
- joint link_LeftHandMiddle3: origin xyz=0 0 0 rpy=0 0 0 -> xyz=0.874827 0.050178 1.43709 rpy=0 0 0
- joint link_LeftHandPinky1: origin xyz=0 0 0 rpy=0 0 0 -> xyz=0.794072 0.087987 1.43272 rpy=0 0 0
- joint link_LeftHandPinky2: origin xyz=0 0 0 rpy=0 0 0 -> xyz=0.830049 0.087987 1.43272 rpy=0 0 0
- joint link_LeftHandPinky3: origin xyz=0 0 0 rpy=0 0 0 -> xyz=0.851314 0.087988 1.43312 rpy=0 0 0
- joint link_LeftHandRing1: origin xyz=0 0 0 rpy=0 0 0 -> xyz=0.804523 0.06889 1.43754 rpy=0 0 0
- joint link_LeftHandRing2: origin xyz=0 0 0 rpy=0 0 0 -> xyz=0.835685 0.068886 1.43714 rpy=0 0 0
- joint link_LeftHandRing3: origin xyz=0 0 0 rpy=0 0 0 -> xyz=0.865221 0.068886 1.43734 rpy=0 0 0
- joint link_LeftHandThumb1: origin xyz=0 0 0 rpy=0 0 0 -> xyz=0.737745 0.02339 1.42165 rpy=0 0 0
- joint link_LeftHandThumb2: origin xyz=0 0 0 rpy=0 0 0 -> xyz=0.770044 0.003941 1.40342 rpy=0 0 0
- joint link_LeftHandThumb3: origin xyz=0 0 0 rpy=0 0 0 -> xyz=0.796849 -0.010757 1.38807 rpy=0 0 0
- joint link_LeftLeg: axis (none) -> 0.000000 0.000000 1.000000; limit (none) -> lower=-3.14 upper=0. effort=1000.0 velocity=0.5; origin xyz=0 0 0 rpy=0 0 0 -> xyz=0.08207 -0.007886 0.529471 rpy=0 0 0; type fixed -> revolute
- joint link_LeftShoulder: origin xyz=0 0 0 rpy=0 0 0 -> xyz=0.04606 0.027266 1.44328 rpy=0 0 0
- joint link_LeftToeBase: axis (none) -> 0.000000 0.000000 1.000000; limit (none) -> lower=-.14 upper=1 effort=1000.0 velocity=0.5; origin xyz=0 0 0 rpy=0 0 0 -> xyz=0.082356 -0.085772 0 rpy=0 0 0; type fixed -> revolute
- joint link_LeftUpLeg: origin xyz=0 0.02076 -1.09271 rpy=0 0 0 -> xyz=0.08208 -0.004943 0.973233 rpy=0 0 0; type fixed -> spherical
- joint link_Neck: limit effort=200.0 velocity=40.0 -> (none); origin xyz=0 0 0 rpy=0 0 0 -> xyz=0 0 1.5 rpy=0 0 0; type floating -> spherical
- joint link_RightArm: origin xyz=0 0 0 rpy=0 0 0 -> xyz=-0.1519 0.0513 1.4367 rpy=0 0 0; type fixed -> spherical
- joint link_RightFoot: origin xyz=0 0 0 rpy=0 0 0 -> xyz=-0.083248 0.021837 0.083976 rpy=0 0 0; type fixed -> spherical
- joint link_RightForeArm: axis (none) -> 0.000000 0.000000 1.000000; limit (none) -> lower=0 upper=3.14 effort=1000.0 velocity=0.5; origin xyz=0 0 0 rpy=0 0 0 -> xyz=-0.4308 0.0513 1.4377 rpy=0 0 0; type fixed -> revolute
- joint link_RightHand: origin xyz=0 0 0 rpy=0 0 0 -> xyz=-0.713253 0.050178 1.43734 rpy=0 0 0; type fixed -> spherical
- joint link_RightHandIndex1: origin xyz=0 0 0 rpy=0 0 0 -> xyz=-0.804532 0.026772 1.43359 rpy=0 0 0
- joint link_RightHandIndex2: origin xyz=0 0 0 rpy=0 0 0 -> xyz=-0.841082 0.027373 1.43234 rpy=0 0 0
- joint link_RightHandIndex3: origin xyz=0 0 0 rpy=0 0 0 -> xyz=-0.869889 0.027973 1.43275 rpy=0 0 0
- joint link_RightHandMiddle1: origin xyz=0 0 0 rpy=0 0 0 -> xyz=-0.808261 0.050178 1.43796 rpy=0 0 0
- joint link_RightHandMiddle2: origin xyz=0 0 0 rpy=0 0 0 -> xyz=-0.845307 0.050178 1.43738 rpy=0 0 0
- joint link_RightHandMiddle3: origin xyz=0 0 0 rpy=0 0 0 -> xyz=-0.874827 0.050178 1.43709 rpy=0 0 0
- joint link_RightHandPinky1: origin xyz=0 0 0 rpy=0 0 0 -> xyz=-0.794072 0.087987 1.43272 rpy=0 0 0
- joint link_RightHandPinky2: origin xyz=0 0 0 rpy=0 0 0 -> xyz=-0.830049 0.087987 1.43272 rpy=0 0 0
- joint link_RightHandPinky3: origin xyz=0 0 0 rpy=0 0 0 -> xyz=-0.851314 0.087988 1.43312 rpy=0 0 0
- joint link_RightHandRing1: origin xyz=0 0 0 rpy=0 0 0 -> xyz=-0.804523 0.06889 1.43754 rpy=0 0 0
- joint link_RightHandRing2: origin xyz=0 0 0 rpy=0 0 0 -> xyz=-0.835685 0.068886 1.43714 rpy=0 0 0
- joint link_RightHandRing3: origin xyz=0 0 0 rpy=0 0 0 -> xyz=-0.865221 0.068886 1.43734 rpy=0 0 0
- joint link_RightHandThumb1: origin xyz=0 0 0 rpy=0 0 0 -> xyz=-0.737745 0.02339 1.42165 rpy=0 0 0
- joint link_RightHandThumb2: origin xyz=0 0 0 rpy=0 0 0 -> xyz=-0.770044 0.003941 1.40342 rpy=0 0 0
- joint link_RightHandThumb3: origin xyz=0 0 0 rpy=0 0 0 -> xyz=-0.796849 -0.010757 1.38807 rpy=0 0 0
- joint link_RightLeg: axis (none) -> 0.000000 0.000000 1.000000; limit (none) -> lower=-3.14 upper=0. effort=1000.0 velocity=0.5; origin xyz=0.08208 0.00477 -1.19426 rpy=0 0 0 -> xyz=-0.08207 -0.007886 0.529471 rpy=0 0 0; type fixed -> revolute
- joint link_RightShoulder: origin xyz=0 0 0 rpy=0 0 0 -> xyz=-0.04606 0.027266 1.44328 rpy=0 0 0
- joint link_RightToeBase: axis (none) -> 0.000000 0.000000 1.000000; limit (none) -> lower=-.14 upper=1 effort=1000.0 velocity=0.5; origin xyz=0 0 0 rpy=0 0 0 -> xyz=-0.082356 -0.085772 0 rpy=0 0 0; type fixed -> revolute
- joint link_RightUpLeg: origin xyz=-0.08208 0.016 0.10154 rpy=0 0 0 -> xyz=-0.08208 -0.004943 0.973233 rpy=0 0 0; type fixed -> spherical
- joint link_Spine1: origin xyz=0 0.01001 0.09618 rpy=0 0 0 -> xyz=0 -0.012 1.2418 rpy=0 0 0; type floating -> spherical
- joint link_Spine2: origin xyz=0 0.01207 -1.28858 rpy=0 0 0 -> xyz=0 0.0015 1.3336 rpy=0 0 0; type floating -> fixed

Commit message: Make all joints fixed

File: urdf/robot.urdf (robot description, URDF)
Before this commit: robot robot, 52 links, 51 joints
Joints:
- joint link_LeftArm: type spherical -> fixed
- joint link_LeftFoot: type spherical -> fixed
- joint link_LeftHand: type spherical -> fixed
- joint link_LeftLeg: type revolute -> fixed
- joint link_LeftUpLeg: type spherical -> fixed
- joint link_Neck: type spherical -> fixed
- joint link_RightArm: type spherical -> fixed
- joint link_RightFoot: type spherical -> fixed
- joint link_RightHand: type spherical -> fixed
- joint link_RightLeg: type revolute -> fixed
- joint link_RightToeBase: type revolute -> fixed
- joint link_RightUpLeg: type spherical -> fixed
- joint link_Spine1: type spherical -> fixed

Commit message: Some edits

File: urdf/robot.urdf (robot description, URDF)
Before this commit: robot robot, 52 links, 51 joints
Joints:
- joint link_Head: origin xyz=0 0 1.6 rpy=1.5708 0 0 -> xyz=7e-05 -0.01698 0.0968 rpy=1.5708 0 0
- joint link_LeftArm: axis (none) -> 1.000000 0.000000 -1.000000; origin xyz=0.1519 0.0513 1.4367 rpy=0 0 0 -> xyz=0.1055 0.02299 -0.00565 rpy=0 0 0; type fixed -> spherical
- joint link_LeftFoot: origin xyz=0.083248 0.021837 0.083976 rpy=0 0 0 -> xyz=0 0 0 rpy=0 0 0; type fixed -> spherical
- joint link_LeftForeArm: axis 0.000000 0.000000 1.000000 -> 0.000000 0.000000 -1.000000; origin xyz=0.4308 0.0513 1.4377 rpy=0 0 0 -> xyz=0.27874 1e-05 0 rpy=0 0 0
- joint link_LeftHand: origin xyz=0.713253 0.050178 1.43734 rpy=0 0 0 -> xyz=0.28308 -0.0001 0 rpy=0 0 0; type fixed -> spherical
- joint link_LeftHandIndex1: origin xyz=0.804532 0.026772 1.43359 rpy=0 0 0 -> xyz=0.09078 -0.02254 -0.0049 rpy=0 0 0
- joint link_LeftHandIndex2: origin xyz=0.841082 0.027373 1.43234 rpy=0 0 0 -> xyz=0.03621 -0.00028 0 rpy=0 0 0
- joint link_LeftHandIndex3: origin xyz=0.869889 0.027973 1.43275 rpy=0 0 0 -> xyz=0.02964 0.00028 -0.0003 rpy=0 0 0
- joint link_LeftHandMiddle1: origin xyz=0.808261 0.050178 1.43796 rpy=0 0 0 -> xyz=0.09542 0.00018 -0.00011 rpy=0 0 0
- joint link_LeftHandMiddle2: origin xyz=0.845307 0.050178 1.43738 rpy=0 0 0 -> xyz=0.03673 -0.00047 0 rpy=0 0 0
- joint link_LeftHandMiddle3: origin xyz=0.874827 0.050178 1.43709 rpy=0 0 0 -> xyz=0.02993 0 0 rpy=0 0 0
- joint link_LeftHandPinky1: origin xyz=0.794072 0.087987 1.43272 rpy=0 0 0 -> xyz=0.08091 0.03815 -0.00528 rpy=0 0 0
- joint link_LeftHandPinky2: origin xyz=0.830049 0.087987 1.43272 rpy=0 0 0 -> xyz=0.03582 0 0.00038 rpy=0 0 0
- joint link_LeftHandPinky3: origin xyz=0.851314 0.087988 1.43312 rpy=0 0 0 -> xyz=0.02092 0 -0.00038 rpy=0 0 0
- joint link_LeftHandRing1: origin xyz=0.804523 0.06889 1.43754 rpy=0 0 0 -> xyz=0.09094 0.01855 -0.00038 rpy=0 0 0
- joint link_LeftHandRing2: origin xyz=0.835685 0.068886 1.43714 rpy=0 0 0 -> xyz=0.03149 0.00018 0 rpy=0 0 0
- joint link_LeftHandRing3: origin xyz=0.865221 0.068886 1.43734 rpy=0 0 0 -> xyz=0.02939 0.0002 -0.00038 rpy=0 0 0
- joint link_LeftHandThumb1: origin xyz=0.737745 0.02339 1.42165 rpy=0 0 0 -> xyz=0.02428 -0.02706 -0.01583 rpy=0 0 0
- joint link_LeftHandThumb2: origin xyz=0.770044 0.003941 1.40342 rpy=0 0 0 -> xyz=0.03265 -0.01871 -0.01922 rpy=0 0 0
- joint link_LeftHandThumb3: origin xyz=0.796849 -0.010757 1.38807 rpy=0 0 0 -> xyz=0.02612 -0.01522 -0.01508 rpy=0 0 0
- joint link_LeftLeg: axis 0.000000 0.000000 1.000000 -> 0.000000 1.000000 0.000000; origin xyz=0.08207 -0.007886 0.529471 rpy=0 0 0 -> xyz=0 0 0 rpy=0 0 0; type fixed -> revolute
- joint link_LeftShoulder: origin xyz=0.04606 0.027266 1.44328 rpy=0 0 0 -> xyz=0.04625 0.02549 0.10964 rpy=0 0 0
- joint link_LeftToeBase: axis 0.000000 0.000000 1.000000 -> 0.000000 1.000000 0.000000; origin xyz=0.082356 -0.085772 0 rpy=0 0 0 -> xyz=0 0 0 rpy=0 0 0
- joint link_LeftUpLeg: axis (none) -> 0.000000 -1.000000 0.000000; limit (none) -> lower=-.14 upper=1 effort=1000.0 velocity=0.5; origin xyz=0.08208 -0.004943 0.973233 rpy=0 0 0 -> xyz=0.00015 0.02076 -1.03935 rpy=0 0 0; type fixed -> revolute
- joint link_Neck: limit (none) -> effort=200.0 velocity=40.0; origin xyz=0 0 1.5 rpy=0 0 0 -> xyz=0.00024 0.02511 0.16549 rpy=0 0 0; type fixed -> spherical
- joint link_RightArm: origin xyz=-0.1519 0.0513 1.4367 rpy=0 0 0 -> xyz=-0.10656 0.02189 -0.00656 rpy=0 0 0; type fixed -> spherical
- joint link_RightFoot: axis (none) -> 0 0 1; limit (none) -> lower=0 upper=3.14 effort=1000.0 velocity=0.5; origin xyz=-0.083248 0.021837 0.083976 rpy=0 0 0 -> xyz=0 0 0 rpy=0 0 0; type fixed -> revolute
- joint link_RightForeArm: axis 0.000000 0.000000 1.000000 -> 0 0 1; limit lower=0 upper=3.14 effort=1000.0 velocity=0.5 -> lower=0 upper=2 effort=1000.0 velocity=0.5; origin xyz=-0.4308 0.0513 1.4377 rpy=0 0 0 -> xyz=-0.2773 0 0.00236 rpy=0 0 0
- joint link_RightHand: origin xyz=-0.713253 0.050178 1.43734 rpy=0 0 0 -> xyz=-0.2841 0 -0.00198 rpy=0 0 0; type fixed -> spherical
- joint link_RightHandIndex1: origin xyz=-0.804532 0.026772 1.43359 rpy=0 0 0 -> xyz=-0.09108 -0.02257 -0.00555 rpy=0 0 0
- joint link_RightHandIndex2: origin xyz=-0.841082 0.027373 1.43234 rpy=0 0 0 -> xyz=-0.03691 0 0.00054 rpy=0 0 0
- joint link_RightHandIndex3: origin xyz=-0.869889 0.027973 1.43275 rpy=0 0 0 -> xyz=-0.02823 -5e-05 0.00027 rpy=0 0 0
- joint link_RightHandMiddle1: origin xyz=-0.808261 0.050178 1.43796 rpy=0 0 0 -> xyz=-0.09542 -5e-05 0.00011 rpy=0 0 0
- joint link_RightHandMiddle2: origin xyz=-0.845307 0.050178 1.43738 rpy=0 0 0 -> xyz=-0.03677 0 0 rpy=0 0 0
- joint link_RightHandMiddle3: origin xyz=-0.874827 0.050178 1.43709 rpy=0 0 0 -> xyz=-0.02945 0 -0.00023 rpy=0 0 0
- joint link_RightHandPinky1: origin xyz=-0.794072 0.087987 1.43272 rpy=0 0 0 -> xyz=-0.08131 0.03814 -0.00471 rpy=0 0 0
- joint link_RightHandPinky2: origin xyz=-0.830049 0.087987 1.43272 rpy=0 0 0 -> xyz=-0.03544 0 9e-05 rpy=0 0 0
- joint link_RightHandPinky3: origin xyz=-0.851314 0.087988 1.43312 rpy=0 0 0 -> xyz=-0.02094 0 -0.00026 rpy=0 0 0
- joint link_RightHandRing1: origin xyz=-0.804523 0.06889 1.43754 rpy=0 0 0 -> xyz=-0.0911 0.01826 -0.00061 rpy=0 0 0
- joint link_RightHandRing2: origin xyz=-0.835685 0.068886 1.43714 rpy=0 0 0 -> xyz=-0.03141 0.00031 0.00031 rpy=0 0 0
- joint link_RightHandRing3: origin xyz=-0.865221 0.068886 1.43734 rpy=0 0 0 -> xyz=-0.02942 0.00031 0 rpy=0 0 0
- joint link_RightHandThumb1: origin xyz=-0.737745 0.02339 1.42165 rpy=0 0 0 -> xyz=-0.02453 -0.02682 -0.01574 rpy=0 0 0
- joint link_RightHandThumb2: origin xyz=-0.770044 0.003941 1.40342 rpy=0 0 0 -> xyz=-0.03242 -0.01872 -0.01836 rpy=0 0 0
- joint link_RightHandThumb3: origin xyz=-0.796849 -0.010757 1.38807 rpy=0 0 0 -> xyz=-0.02676 -0.01543 -0.01549 rpy=0 0 0
- joint link_RightLeg: origin xyz=-0.08207 -0.007886 0.529471 rpy=0 0 0 -> xyz=0.08208 0.00477 -1.19426 rpy=0 0 0; type fixed -> revolute
- joint link_RightShoulder: origin xyz=-0.04606 0.027266 1.44328 rpy=0 0 0 -> xyz=-0.04536 0.02663 0.10998 rpy=0 0 0
- joint link_RightToeBase: origin xyz=-0.082356 -0.085772 0 rpy=0 0 0 -> xyz=0 0 0 rpy=0 0 0; type fixed -> revolute
- joint link_RightUpLeg: origin xyz=-0.08208 -0.004943 0.973233 rpy=0 0 0 -> xyz=-0.08193 0.01599 0.15491 rpy=0 0 0; type fixed -> spherical
- joint link_Spine: origin xyz=0 -0.00132 0.09968 rpy=0 0 0 -> xyz=0.00037 -0.00172 0.10244 rpy=0 0 0
- joint link_Spine1: origin xyz=0 -0.012 1.2418 rpy=0 0 0 -> xyz=-0.00026 0.01027 0.10076 rpy=0 0 0; type fixed -> spherical
- joint link_Spine2: origin xyz=0 0.0015 1.3336 rpy=0 0 0 -> xyz=0 0.01405 0.09109 rpy=0 0 0
