Commit message: Fix robot.urdf, add examples

File: urdf/robot.urdf (robot description, URDF)
Before this commit: robot robot, 52 links, 51 joints
Links:
- link link_LeftHandThumb1: geometry collision mesh filename=c_LeftHandThumb1.stl scale=1.0 1.0 1.0; collision sphere radius=0.01773
- link link_LeftHandThumb2: geometry collision mesh filename=c_LeftHandThumb2.stl scale=0.01 0.01 0.01; collision sphere radius=0.01069
- link link_LeftHandThumb3: geometry collision mesh filename=c_LeftHandThumb3.stl scale=1.0 1.0 1.0; collision sphere radius=0.00798
- link link_RightHandThumb2: geometry collision mesh filename=c_RightHandThumb2.stl scale=1.0 1.0 1.0; collision sphere radius=0.01094
- link link_RightHandThumb3: geometry collision mesh filename=c_RightHandThumb3.stl scale=1.0 1.0 1.0; collision sphere radius=0.00816
Joints:
- joint link_LeftArm: axis 1.000000 0.000000 -1.000000 -> 0.000000 1.000000 0.000000; limit (none) -> lower=-2 upper=2 effort=1000.0 velocity=0.5; type spherical -> revolute
- joint link_LeftFoot: axis (none) -> -1 0 0; limit (none) -> lower=0 upper=3.14 effort=1000.0 velocity=0.5; origin xyz=0 0 0 rpy=0 0 0 -> xyz=0 0.0304 -0.4433 rpy=0 0 0; type spherical -> revolute
- joint link_LeftHand: type spherical -> fixed
- joint link_LeftLeg: axis 0.000000 1.000000 0.000000 -> -1.000000 0.000000 0.000000; limit lower=-3.14 upper=0. effort=1000.0 velocity=0.5 -> lower=-2 upper=0. effort=1000.0 velocity=0.5; origin xyz=0 0 0 rpy=0 0 0 -> xyz=0 -0.00269 -0.44503 rpy=0 0 0
- joint link_LeftShoulder: axis (none) -> -1.000000 0.000000 0.000000; limit (none) -> lower=-2 upper=0. effort=1000.0 velocity=0.5; type fixed -> revolute
- joint link_LeftToeBase: origin xyz=0 0 0 rpy=0 0 0 -> xyz=0.00065 -0.10737 -0.06079 rpy=0 0 0
- joint link_LeftUpLeg: axis 0.000000 -1.000000 0.000000 -> 1.000000 1.000000 0.000000; origin xyz=0.00015 0.02076 -1.03935 rpy=0 0 0 -> xyz=0.08245 0.01519 -0.06714 rpy=0 0 0; type revolute -> spherical
- joint link_Neck: axis (none) -> 1.000000 1.000000 0.000000
- joint link_RightArm: axis (none) -> 0.000000 1.000000 0.000000; limit (none) -> lower=-2 upper=2 effort=1000.0 velocity=0.5; type spherical -> revolute
- joint link_RightFoot: axis 0 0 1 -> -1 0 0; limit lower=0 upper=3.14 effort=1000.0 velocity=0.5 -> lower=-1 upper=1 effort=1000.0 velocity=0.5; origin xyz=0 0 0 rpy=0 0 0 -> xyz=-0.00065 0.03005 -0.44359 rpy=0 0 0
- joint link_RightHand: type spherical -> fixed
- joint link_RightLeg: axis 0.000000 0.000000 1.000000 -> -1.000000 0.000000 0.000000; limit lower=-3.14 upper=0. effort=1000.0 velocity=0.5 -> lower=-2 upper=0. effort=1000.0 velocity=0.5; origin xyz=0.08208 0.00477 -1.19426 rpy=0 0 0 -> xyz=0.00065 -0.00196 -0.44457 rpy=0 0 0
- joint link_RightShoulder: axis (none) -> -1.000000 0.000000 0.000000; limit (none) -> lower=-2 upper=0. effort=1000.0 velocity=0.5; type fixed -> revolute
- joint link_RightToeBase: origin xyz=0 0 0 rpy=0 0 0 -> xyz=0 -0.11037 -0.06152 rpy=0 0 0
- joint link_RightUpLeg: axis (none) -> 1.000000 1.000000 1.000000; origin xyz=-0.08193 0.01599 0.15491 rpy=0 0 0 -> xyz=-0.08209 0.01519 -0.06714 rpy=0 0 0
- joint link_Spine1: axis (none) -> 1.000000 1.000000 1.000000

Commit message: Fix urdf joint configs

File: urdf/robot.urdf (robot description, URDF)
Before this commit: robot robot, 52 links, 51 joints
Joints:
- joint link_LeftFoot: axis -1 0 0 -> 1 0 0
- joint link_LeftLeg: limit lower=-2 upper=0. effort=1000.0 velocity=0.5 -> lower=-2.5 upper=0 effort=1000.0 velocity=0.5
- joint link_LeftShoulder: axis -1.000000 0.000000 0.000000 -> 0.000000 1.000000 0.000000; limit lower=-2 upper=0. effort=1000.0 velocity=0.5 -> lower=0 upper=0.2 effort=1000.0 velocity=0.5
- joint link_LeftToeBase: axis 0.000000 1.000000 0.000000 -> 1.000000 0.000000 0.000000; limit lower=-.14 upper=1 effort=1000.0 velocity=0.5 -> lower=-0.6 upper=0.6 effort=1000.0 velocity=0.5
- joint link_LeftUpLeg: axis 1.000000 1.000000 0.000000 -> 1.000000 1.000000 1.000000
- joint link_RightArm: type revolute -> spherical
- joint link_RightFoot: axis -1 0 0 -> 1 0 0; limit lower=-1 upper=1 effort=1000.0 velocity=0.5 -> lower=-0.6 upper=0.4 effort=1000.0 velocity=0.5
- joint link_RightLeg: limit lower=-2 upper=0. effort=1000.0 velocity=0.5 -> lower=-2.5 upper=0 effort=1000.0 velocity=0.5
- joint link_RightShoulder: axis -1.000000 0.000000 0.000000 -> 0.000000 1.000000 0.000000; limit lower=-2 upper=0. effort=1000.0 velocity=0.5 -> lower=0 upper=0.2 effort=1000.0 velocity=0.5
- joint link_RightToeBase: axis 0.000000 0.000000 1.000000 -> 1.000000 0.000000 0.000000; limit lower=-.14 upper=1 effort=1000.0 velocity=0.5 -> lower=-0.6 upper=0.6 effort=1000.0 velocity=0.5
- joint link_RightUpLeg: limit (none) -> lower=-.14 upper=1 effort=1000.0 velocity=0.5

Commit message: Fix collision objects, add examples

File: urdf/robot.urdf (robot description, URDF)
Before this commit: robot robot, 52 links, 51 joints
Links:
- link link_LeftForeArm: geometry collision mesh filename=c_LeftForeArm.stl scale=1.0 1.0 1.0; collision sphere radius=0.04142
- link link_LeftHand: geometry collision mesh filename=c_LeftHand.stl scale=1.0 1.0 1.0; collision sphere radius=0.02982
- link link_LeftHandIndex1: geometry collision mesh filename=c_LeftHandIndex.stl scale=1.0 1.0 1.0; collision sphere radius=0.01204
- link link_LeftHandIndex2: geometry collision mesh filename=c_LeftHandIndex2.stl scale=1.0 1.0 1.0; collision sphere radius=0.00977
- link link_LeftHandIndex3: geometry collision mesh filename=c_LeftHandIndex3.stl scale=1.0 1.0 1.0; collision sphere radius=0.00859
- link link_LeftHandMiddle1: geometry collision mesh filename=c_LeftHandMiddle1.stl scale=1.0 1.0 1.0; collision sphere radius=0.01297
- link link_LeftHandMiddle2: geometry collision mesh filename=c_LeftHandMiddle2.stl scale=1.0 1.0 1.0; collision sphere radius=0.00975
- link link_LeftHandMiddle3: geometry collision mesh filename=c_LeftHandMiddle3.stl scale=1.0 1.0 1.0; collision sphere radius=0.00831
- link link_LeftHandPinky1: geometry collision mesh filename=c_LeftHandPinky1.stl scale=1.0 1.0 1.0; collision sphere radius=0.01219
- link link_LeftHandPinky2: geometry collision mesh filename=c_LeftHandPinky2.stl scale=1.0 1.0 1.0; collision sphere radius=0.00827
- link link_LeftHandPinky3: geometry collision mesh filename=c_LeftHandPinky3.stl scale=1.0 1.0 1.0; collision sphere radius=0.0071
- link link_LeftHandRing1: geometry collision mesh filename=c_LeftHandRing1.stl scale=1.0 1.0 1.0; collision sphere radius=0.01255
- link link_LeftHandRing2: geometry collision mesh filename=c_LeftHandRing2.stl scale=1.0 1.0 1.0; collision sphere radius=0.00966
- link link_LeftHandRing3: geometry collision mesh filename=c_LeftHandRing3.stl scale=1.0 1.0 1.0; collision sphere radius=0.0085
- link link_LeftLeg: geometry collision mesh filename=c_LeftLeg.stl scale=1.0 1.0 1.0; collision sphere radius=0.06134
- link link_LeftUpLeg: geometry collision mesh filename=c_LeftUpLeg.stl scale=1.0 1.0 1.0; collision sphere radius=0.1245
- link link_RightForeArm: geometry collision mesh filename=c_RightForeArm.stl scale=1.0 1.0 1.0; collision sphere radius=0.03853
- link link_RightHand: geometry collision mesh filename=c_RightHand.stl scale=1.0 1.0 1.0; collision sphere radius=0.02982
- link link_RightHandIndex1: geometry collision mesh filename=c_RightHandIndex1.stl scale=1.0 1.0 1.0; collision sphere radius=0.01204
- link link_RightHandIndex2: geometry collision mesh filename=c_RightHandIndex2.stl scale=1.0 1.0 1.0; collision sphere radius=0.00977
- link link_RightHandIndex3: geometry collision mesh filename=c_RightHandIndex3.stl scale=1.0 1.0 1.0; collision sphere radius=0.00859
- link link_RightHandMiddle1: geometry collision mesh filename=c_RightHandMiddle1.stl scale=1.0 1.0 1.0; collision sphere radius=0.01297
- link link_RightHandMiddle2: geometry collision mesh filename=c_RightHandMiddle2.stl scale=1.0 1.0 1.0; collision sphere radius=0.00975
- link link_RightHandMiddle3: geometry collision mesh filename=c_RightHandMiddle3.stl scale=1.0 1.0 1.0; collision sphere radius=0.00831
- link link_RightHandPinky1: geometry collision mesh filename=c_RightHandPinky1.stl scale=1.0 1.0 1.0; collision sphere radius=0.01219
- link link_RightHandPinky2: geometry collision mesh filename=c_RightHandPinky2.stl scale=1.0 1.0 1.0; collision sphere radius=0.00827
- link link_RightHandPinky3: geometry collision mesh filename=c_RightHandPinky3.stl scale=1.0 1.0 1.0; collision sphere radius=0.0071
- link link_RightHandRing1: geometry collision mesh filename=c_RightHandRing1.stl scale=1.0 1.0 1.0; collision sphere radius=0.01255
- link link_RightHandRing2: geometry collision mesh filename=c_RightHandRing2.stl scale=1.0 1.0 1.0; collision sphere radius=0.00966
- link link_RightHandRing3: geometry collision mesh filename=c_RightHandRing3.stl scale=1.0 1.0 1.0; collision sphere radius=0.0085
- link link_RightHandThumb1: geometry collision mesh filename=c_RightHandThumb1.stl scale=1.0 1.0 1.0; collision sphere radius=0.01832
- link link_RightLeg: geometry collision mesh filename=c_RightLeg.stl scale=1.0 1.0 1.0; collision sphere radius=0.06158
- link link_RightUpLeg: geometry collision mesh filename=c_RightUpLeg.stl scale=1.0 1.0 1.0; collision sphere radius=0.08656
- link link_Spine: geometry collision sphere radius=0.12974; visual mesh filename=Spine.stl scale=1.0 1.0 1.0
Joints:
- joint link_LeftArm: type revolute -> spherical
- joint link_LeftShoulder: type revolute -> fixed
- joint link_RightShoulder: type revolute -> fixed
- joint link_Spine2: type fixed -> spherical

Commit message: Fix robot.urdf

File: urdf/robot.urdf (robot description, URDF)
Before this commit: robot robot, 52 links, 51 joints
Joints:
- joint link_Head: limit lower=-4.0 upper=4.0 effort=500.0 velocity=40.0 -> lower=-1.6 upper=1.6 effort=10.0 velocity=10.0
- joint link_LeftArm: limit lower=-2 upper=2 effort=1000.0 velocity=0.5 -> lower=-2 upper=2 effort=1000.0 velocity=10
- joint link_LeftFoot: limit lower=0 upper=3.14 effort=1000.0 velocity=0.5 -> lower=-0.6 upper=0.4 effort=10.0 velocity=10
- joint link_LeftForeArm: axis 0.000000 0.000000 -1.000000 -> 0 0 1; limit lower=0 upper=3.14 effort=1000.0 velocity=0.5 -> lower=0 upper=2 effort=1.0 velocity=10
- joint link_LeftLeg: axis -1.000000 0.000000 0.000000 -> 1.000000 0.000000 0.000000; limit lower=-2.5 upper=0 effort=1000.0 velocity=0.5 -> lower=0 upper=2.5 effort=10.0 velocity=10
- joint link_LeftShoulder: limit lower=0 upper=0.2 effort=1000.0 velocity=0.5 -> lower=0 upper=0.2 effort=1000.0 velocity=10
- joint link_LeftToeBase: limit lower=-0.6 upper=0.6 effort=1000.0 velocity=0.5 -> lower=-0.6 upper=0.6 effort=10.0 velocity=10
- joint link_LeftUpLeg: limit lower=-.14 upper=1 effort=1000.0 velocity=0.5 -> lower=-.14 upper=1 effort=1000.0 velocity=10
- joint link_RightArm: limit lower=-2 upper=2 effort=1000.0 velocity=0.5 -> lower=-2 upper=2 effort=1000.0 velocity=10
- joint link_RightFoot: limit lower=-0.6 upper=0.4 effort=1000.0 velocity=0.5 -> lower=-0.6 upper=0.4 effort=10.0 velocity=10
- joint link_RightForeArm: limit lower=0 upper=2 effort=1000.0 velocity=0.5 -> lower=0 upper=2 effort=1.0 velocity=10
- joint link_RightLeg: axis -1.000000 0.000000 0.000000 -> 1.000000 0.000000 0.000000; limit lower=-2.5 upper=0 effort=1000.0 velocity=0.5 -> lower=0 upper=2.5 effort=10.0 velocity=10
- joint link_RightShoulder: limit lower=0 upper=0.2 effort=1000.0 velocity=0.5 -> lower=0 upper=0.2 effort=1000.0 velocity=10
- joint link_RightToeBase: limit lower=-0.6 upper=0.6 effort=1000.0 velocity=0.5 -> lower=-0.6 upper=0.6 effort=10.0 velocity=10
- joint link_RightUpLeg: limit lower=-.14 upper=1 effort=1000.0 velocity=0.5 -> lower=-.14 upper=1 effort=1000.0 velocity=10
- joint link_Spine1: limit effort=500.0 velocity=40.0 -> effort=10.0 velocity=10.0
- joint link_Spine2: axis (none) -> 1.000000 1.000000 1.000000; limit effort=200.0 velocity=40.0 -> effort=10.0 velocity=10.0

Commit message: Make hands movable

File: urdf/robot.urdf (robot description, URDF)
Before this commit: robot robot, 52 links, 51 joints
Joints:
- joint link_LeftHand: axis (none) -> 1 1 0; type fixed -> spherical
- joint link_LeftHandIndex1: axis (none) -> 1 0 0; limit (none) -> lower=0 upper=2 effort=1.0 velocity=10; type fixed -> revolute
- joint link_LeftHandIndex2: axis (none) -> 1 0 0; limit (none) -> lower=0 upper=2 effort=1.0 velocity=10; type fixed -> revolute
- joint link_LeftHandIndex3: axis (none) -> 1 0 0; limit (none) -> lower=0 upper=2 effort=1.0 velocity=10; type fixed -> revolute
- joint link_LeftHandMiddle1: axis (none) -> 1 0 0; limit (none) -> lower=0 upper=2 effort=1.0 velocity=10; type fixed -> revolute
- joint link_LeftHandMiddle2: axis (none) -> 1 0 0; limit (none) -> lower=0 upper=2 effort=1.0 velocity=10; type fixed -> revolute
- joint link_LeftHandMiddle3: axis (none) -> 1 0 0; limit (none) -> lower=0 upper=2 effort=1.0 velocity=10; type fixed -> revolute
- joint link_LeftHandPinky1: axis (none) -> 1 0 0; limit (none) -> lower=0 upper=2 effort=1.0 velocity=10; type fixed -> revolute
- joint link_LeftHandPinky2: axis (none) -> 1 0 0; limit (none) -> lower=0 upper=2 effort=1.0 velocity=10; type fixed -> revolute
- joint link_LeftHandPinky3: axis (none) -> 1 0 0; limit (none) -> lower=0 upper=2 effort=1.0 velocity=10; type fixed -> revolute
- joint link_LeftHandRing1: axis (none) -> 1 0 0; limit (none) -> lower=0 upper=2 effort=1.0 velocity=10; type fixed -> revolute
- joint link_LeftHandRing2: axis (none) -> 1 0 0; limit (none) -> lower=0 upper=2 effort=1.0 velocity=10; type fixed -> revolute
- joint link_LeftHandRing3: axis (none) -> 1 0 0; limit (none) -> lower=0 upper=2 effort=1.0 velocity=10; type fixed -> revolute
- joint link_LeftHandThumb1: axis (none) -> 0.5 0 0.5; limit (none) -> lower=0 upper=2 effort=1.0 velocity=10; type fixed -> revolute
- joint link_LeftHandThumb2: axis (none) -> 0.5 0 0.5; limit (none) -> lower=0 upper=2 effort=1.0 velocity=10; type fixed -> revolute
- joint link_LeftHandThumb3: axis (none) -> 0.5 0 0.5; limit (none) -> lower=0 upper=2 effort=1.0 velocity=10; type fixed -> revolute
- joint link_RightHand: axis (none) -> 1 1 0; type fixed -> spherical
- joint link_RightHandIndex1: axis (none) -> 1 0 0; limit (none) -> lower=0 upper=2 effort=1.0 velocity=10; type fixed -> revolute
- joint link_RightHandIndex2: axis (none) -> 1 0 0; limit (none) -> lower=0 upper=2 effort=1.0 velocity=10; type fixed -> revolute
- joint link_RightHandIndex3: axis (none) -> 1 0 0; limit (none) -> lower=0 upper=2 effort=1.0 velocity=10; type fixed -> revolute
- joint link_RightHandMiddle1: axis (none) -> 1 0 0; limit (none) -> lower=0 upper=2 effort=1.0 velocity=10; type fixed -> revolute
- joint link_RightHandMiddle2: axis (none) -> 1 0 0; limit (none) -> lower=0 upper=2 effort=1.0 velocity=10; type fixed -> revolute
- joint link_RightHandMiddle3: axis (none) -> 1 0 0; limit (none) -> lower=0 upper=2 effort=1.0 velocity=10; type fixed -> revolute
- joint link_RightHandPinky1: axis (none) -> 1 0 0; limit (none) -> lower=0 upper=2 effort=1.0 velocity=10; type fixed -> revolute
- joint link_RightHandPinky2: axis (none) -> 1 0 0; limit (none) -> lower=0 upper=2 effort=1.0 velocity=10; type fixed -> revolute
- joint link_RightHandPinky3: axis (none) -> 1 0 0; limit (none) -> lower=0 upper=2 effort=1.0 velocity=10; type fixed -> revolute
- joint link_RightHandRing1: axis (none) -> 1 0 0; limit (none) -> lower=0 upper=2 effort=1.0 velocity=10; type fixed -> revolute
- joint link_RightHandRing2: axis (none) -> 1 0 0; limit (none) -> lower=0 upper=2 effort=1.0 velocity=10; type fixed -> revolute
- joint link_RightHandRing3: axis (none) -> 1 0 0; limit (none) -> lower=0 upper=2 effort=1.0 velocity=10; type fixed -> revolute
- joint link_RightHandThumb1: type fixed -> spherical
- joint link_RightHandThumb2: axis (none) -> 0.5 0 0.5; limit (none) -> lower=0 upper=2 effort=1.0 velocity=10; type fixed -> revolute
- joint link_RightHandThumb3: axis (none) -> 0.5 0 0.5; limit (none) -> lower=0 upper=2 effort=1.0 velocity=10; type fixed -> revolute

Commit message: Some changes for debug

File: urdf/robot.urdf (robot description, URDF)
Before this commit: robot robot, 52 links, 51 joints
Joints:
- joint link_LeftHandIndex1: axis 1 0 0 -> 0 1 0; limit lower=0 upper=2 effort=1.0 velocity=10 -> lower=0 upper=1.5 effort=1.0 velocity=10
- joint link_LeftHandIndex2: axis 1 0 0 -> 0 1 0; limit lower=0 upper=2 effort=1.0 velocity=10 -> lower=0 upper=1.5 effort=1.0 velocity=10
- joint link_LeftHandIndex3: axis 1 0 0 -> 0 1 0; limit lower=0 upper=2 effort=1.0 velocity=10 -> lower=0 upper=1.5 effort=1.0 velocity=10
- joint link_LeftHandMiddle1: axis 1 0 0 -> 0 1 0; limit lower=0 upper=2 effort=1.0 velocity=10 -> lower=0 upper=1.5 effort=1.0 velocity=10
- joint link_LeftHandMiddle2: axis 1 0 0 -> 0 1 0; limit lower=0 upper=2 effort=1.0 velocity=10 -> lower=0 upper=1.5 effort=1.0 velocity=10
- joint link_LeftHandMiddle3: axis 1 0 0 -> 0 1 0; limit lower=0 upper=2 effort=1.0 velocity=10 -> lower=0 upper=1.5 effort=1.0 velocity=10
- joint link_LeftHandPinky1: axis 1 0 0 -> 0 1 0; limit lower=0 upper=2 effort=1.0 velocity=10 -> lower=0 upper=1.5 effort=1.0 velocity=10
- joint link_LeftHandPinky2: axis 1 0 0 -> 0 1 0; limit lower=0 upper=2 effort=1.0 velocity=10 -> lower=0 upper=1.5 effort=1.0 velocity=10
- joint link_LeftHandPinky3: axis 1 0 0 -> 0 1 0; limit lower=0 upper=2 effort=1.0 velocity=10 -> lower=0 upper=1.5 effort=1.0 velocity=10
- joint link_LeftHandRing1: axis 1 0 0 -> 0 1 0; limit lower=0 upper=2 effort=1.0 velocity=10 -> lower=0 upper=1.5 effort=1.0 velocity=10
- joint link_LeftHandRing2: axis 1 0 0 -> 0 1 0; limit lower=0 upper=2 effort=1.0 velocity=10 -> lower=0 upper=1.5 effort=1.0 velocity=10
- joint link_LeftHandRing3: axis 1 0 0 -> 0 1 0; limit lower=0 upper=2 effort=1.0 velocity=10 -> lower=0 upper=1.5 effort=1.0 velocity=10
- joint link_LeftHandThumb1: limit lower=0 upper=2 effort=1.0 velocity=10 -> lower=0 upper=1.5 effort=1.0 velocity=10
- joint link_LeftHandThumb2: axis 0.5 0 0.5 -> -0.05 -0.2 0.1; limit lower=0 upper=2 effort=1.0 velocity=10 -> lower=0 upper=1.5 effort=10.0 velocity=10
- joint link_LeftHandThumb3: axis 0.5 0 0.5 -> -0.05 -0.2 0.1; limit lower=0 upper=2 effort=1.0 velocity=10 -> lower=0 upper=1 effort=10.0 velocity=10
- joint link_RightHandIndex1: axis 1 0 0 -> 0 -1 0; limit lower=0 upper=2 effort=1.0 velocity=10 -> lower=0 upper=1.5 effort=1.0 velocity=10
- joint link_RightHandIndex2: axis 1 0 0 -> 0 -1 0; limit lower=0 upper=2 effort=1.0 velocity=10 -> lower=0 upper=1.5 effort=1.0 velocity=10
- joint link_RightHandIndex3: axis 1 0 0 -> 0 -1 0; limit lower=0 upper=2 effort=1.0 velocity=10 -> lower=0 upper=1.5 effort=1.0 velocity=10
- joint link_RightHandMiddle1: axis 1 0 0 -> 0 -1 0; limit lower=0 upper=2 effort=1.0 velocity=10 -> lower=0 upper=1.5 effort=1.0 velocity=10
- joint link_RightHandMiddle2: axis 1 0 0 -> 0 -1 0; limit lower=0 upper=2 effort=1.0 velocity=10 -> lower=0 upper=1.5 effort=1.0 velocity=10
- joint link_RightHandMiddle3: axis 1 0 0 -> 0 -1 0; limit lower=0 upper=2 effort=1.0 velocity=10 -> lower=0 upper=1.5 effort=1.0 velocity=10
- joint link_RightHandPinky1: axis 1 0 0 -> 0 -1 0; limit lower=0 upper=2 effort=1.0 velocity=10 -> lower=0 upper=1.5 effort=1.0 velocity=10
- joint link_RightHandPinky2: axis 1 0 0 -> 0 -1 0; limit lower=0 upper=2 effort=1.0 velocity=10 -> lower=0 upper=1.5 effort=1.0 velocity=10
- joint link_RightHandPinky3: axis 1 0 0 -> 0 -1 0; limit lower=0 upper=2 effort=1.0 velocity=10 -> lower=0 upper=1.5 effort=1.0 velocity=10
- joint link_RightHandRing1: axis 1 0 0 -> 0 -1 0; limit lower=0 upper=2 effort=1.0 velocity=10 -> lower=0 upper=1.5 effort=1.0 velocity=10
- joint link_RightHandRing2: axis 1 0 0 -> 0 -1 0; limit lower=0 upper=2 effort=1.0 velocity=10 -> lower=0 upper=1.5 effort=1.0 velocity=10
- joint link_RightHandRing3: axis 1 0 0 -> 0 -1 0; limit lower=0 upper=2 effort=1.0 velocity=10 -> lower=0 upper=1.5 effort=1.0 velocity=10
- joint link_RightHandThumb1: axis (none) -> 1 0 1
- joint link_RightHandThumb2: axis 0.5 0 0.5 -> 0.05 -0.2 0.1; limit lower=0 upper=2 effort=1.0 velocity=10 -> lower=0 upper=1.5 effort=10.0 velocity=10
- joint link_RightHandThumb3: axis 0.5 0 0.5 -> 0.05 -0.2 0.1; limit lower=0 upper=2 effort=1.0 velocity=10 -> lower=0 upper=1 effort=10.0 velocity=10
