Commit message: Current status

File: urdf/robot_no_hands.urdf (robot description, URDF)
Before this commit: robot robot, 22 links, 21 joints
Links:
- link link_LeftArm: geometry collision mesh filename=c_LeftArm.stl scale=1.0 1.0 1.0; collision sphere radius=0.04861
- link link_LeftShoulder: geometry 
- link link_RightArm: geometry collision mesh filename=c_RightArm.stl scale=1.0 1.0 1.0; collision sphere radius=0.04861
- link link_RightShoulder: geometry 
Joints:
- joint link_LeftArm: origin xyz=0.1055 0.02299 -0.00565 rpy=0 0 0 -> xyz=0.10592 0.02232 -0.00525 rpy=0 0 0
- joint link_LeftForeArm: origin xyz=0.27874 1e-05 0 rpy=0 0 0 -> xyz=0.27842 0 0 rpy=0 0 0
- joint link_LeftHand: origin xyz=0.28308 -0.0001 0 rpy=0 0 0 -> xyz=0.28349 -0.00079 -0.00016 rpy=0 0 0; type fixed -> spherical
- joint link_LeftLeg: axis 1.000000 0.000000 0.000000 -> 0 0 1; origin xyz=0 -0.00269 -0.44503 rpy=0 0 0 -> xyz=0.00023 -0.00426 -0.44522 rpy=0 0 0
- joint link_LeftShoulder: axis 0.000000 1.000000 0.000000 -> 1 0 0; limit lower=0 upper=0.2 effort=1000.0 velocity=10 -> lower=-1 upper=2 effort=1000.0 velocity=10; origin xyz=0.04625 0.02549 0.10964 rpy=0 0 0 -> xyz=0.0457 0.02671 0.10946 rpy=0 0 0
- joint link_LeftToeBase: origin xyz=0.00065 -0.10737 -0.06079 rpy=0 0 0 -> xyz=-0.00023 -0.08629 -0.08665 rpy=0 0 0
- joint link_LeftUpLeg: axis 1.000000 1.000000 1.000000 -> 0 0 105; limit lower=-.14 upper=1 effort=1000.0 velocity=10 -> lower=-4 upper=4 effort=1000.0 velocity=10; origin xyz=0.08245 0.01519 -0.06714 rpy=0 0 0 -> xyz=0.08208 0.016 0.9724 rpy=0 0 0
- joint link_Neck: origin xyz=0.00024 0.02511 0.16549 rpy=0 0 0 -> xyz=0.00019 0.02495 0.16556 rpy=0 0 0
- joint link_RightArm: origin xyz=-0.10656 0.02189 -0.00656 rpy=0 0 0 -> xyz=-0.10593 0.02232 -0.00525 rpy=0 0 0
- joint link_RightForeArm: origin xyz=-0.2773 0 0.00236 rpy=0 0 0 -> xyz=-0.27841 0 0 rpy=0 0 0
- joint link_RightHand: origin xyz=-0.2841 0 -0.00198 rpy=0 0 0 -> xyz=-0.28332 -0.00066 -0.00035 rpy=0 0 0; type fixed -> spherical
- joint link_RightShoulder: axis 0.000000 1.000000 0.000000 -> -1 0 0; origin xyz=-0.04536 0.02663 0.10998 rpy=0 0 0 -> xyz=-0.0457 0.02671 0.10946 rpy=0 0 0
- joint link_RightUpLeg: origin xyz=-0.08209 0.01519 -0.06714 rpy=0 0 0 -> xyz=-0.08224 -0.00557 0.9722 rpy=0 0 0
- joint link_Spine: origin xyz=0.00037 -0.00172 0.10244 rpy=0 0 0 -> xyz=0.00022 -0.00248 1.14179 rpy=0 0 0
- joint link_Spine1: origin xyz=-0.00026 0.01027 0.10076 rpy=0 0 0 -> xyz=-0.00022 0.01148 0.10078 rpy=0 0 0
- joint link_Spine2: origin xyz=0 0.01405 0.09109 rpy=0 0 0 -> xyz=0 0.013 0.091 rpy=0 0 0
