Commit message: Implement OD robot

File: quadruped_envs/urdf/od.urdf (robot description, URDF)
Before this commit: robot od, 13 links, 12 joints
Links:
- added link imu_link, mass 0.001; collision box size=.001 .001 .001; visual box size=0.001 0.001 0.001
Joints:
- added joint imu_joint: type fixed, parent link_root, child imu_link, origin xyz=0 0 0 rpy=0 0 0
- joint link_l_leg_d: limit lower=-1.31 upper=2.443 effort=2.7 velocity=50.0 -> lower=-6.3 upper=6.3 effort=2.7 velocity=50.0

Commit message: Fix urdf issues

File: quadruped_envs/urdf/od.urdf (robot description, URDF)
Before this commit: robot od, 14 links, 13 joints
Links:
- link link_hip_a: geometry collision box size=0.1759 0.0389 0.04438; visual mesh filename=HipFeModuleA.stl scale=1.0 1.0 1.0
- link link_hip_b: geometry collision box size=0.201 0.0389 0.04438; visual mesh filename=HipAdapterB.stl scale=1.0 1.0 1.0
- link link_hip_c: geometry collision box size=0.201 0.0389 0.04438; visual mesh filename=HipAdapterC.stl scale=1.0 1.0 1.0
- link link_hip_d: geometry collision box size=0.1759 0.0389 0.04438; visual mesh filename=HipFeModuleD.stl scale=1.0 1.0 1.0
- link link_l_leg_a: geometry collision box size=0.09247 0.0085 0.10287; collision cylinder length=0.032 radius=0.016
- link link_l_leg_b: geometry collision box size=0.09247 0.0085 0.10287; collision cylinder length=0.032 radius=0.016
- link link_l_leg_c: geometry collision box size=0.09367 0.0085 0.10182; collision cylinder length=0.03188 radius=0.01594
- link link_l_leg_d: geometry collision box size=0.09247 0.0085 0.10287; collision cylinder length=0.032 radius=0.016
- link link_root: geometry collision box size=0.01 0.04 0.04; collision box size=0.01 0.04 0.04
- link link_u_leg_a: geometry collision box size=0.11331 0.014 0.12771; collision cylinder length=0.035 radius=0.0175
- link link_u_leg_b: geometry collision box size=0.11331 0.014 0.12771; collision cylinder length=0.035 radius=0.0175
- link link_u_leg_c: geometry collision box size=0.11331 0.014 0.12771; collision cylinder length=0.035 radius=0.0175
- link link_u_leg_d: geometry collision box size=0.11331 0.014 0.12771; collision cylinder length=0.035 radius=0.0175
Joints:
- joint link_hip_a: origin xyz=-0.1939 -0.09 0.3 rpy=0 0 0 -> xyz=-0.1939 -0.09 0 rpy=0 0 0
- joint link_hip_b: origin xyz=-0.1939 0.09 0.3 rpy=0 0 0 -> xyz=-0.1939 0.09 0 rpy=0 0 0
- joint link_hip_c: origin xyz=0.1939 -0.09 0.3 rpy=0 0 0 -> xyz=0.1939 -0.09 0 rpy=0 0 0
- joint link_hip_d: origin xyz=0.1939 0.09 0.3 rpy=0 0 0 -> xyz=0.1939 0.09 0 rpy=0 0 0
- joint link_l_leg_a: origin xyz=0.10113 -0.05695 -0.12354 rpy=0 -2.83267 0 -> xyz=0.10112 -0.05695 -0.12354 rpy=0 0 0
- joint link_l_leg_b: origin xyz=0.10113 0.05695 -0.12354 rpy=0 -2.82743 0 -> xyz=0.10112 0.05695 -0.12354 rpy=0 0 0
- joint link_l_leg_c: origin xyz=-0.10113 -0.05695 -0.12354 rpy=0 0 0 -> xyz=0.09841 -0.05695 -0.12588 rpy=0 0 0
- joint link_l_leg_d: origin xyz=-0.10112 0.05695 -0.12354 rpy=0 0 0 -> xyz=0.09841 0.05695 -0.12588 rpy=0 -1.34948 0
- joint link_u_leg_a: origin xyz=0 0 0 rpy=0 1.37881 0 -> xyz=0 0 0 rpy=0 0 0
- joint link_u_leg_b: origin xyz=0 0 0 rpy=0 1.37881 0 -> xyz=0 0 0 rpy=0 0 0

Commit message: Fix urdf issues

File: quadruped_envs/urdf/od.urdf (robot description, URDF)
Before this commit: robot od, 14 links, 13 joints
Links:
- link link_l_leg_a: geometry collision mesh filename=collision_LowerLegA.stl scale=1.0 1.0 1.0; visual mesh filename=LowerLegA.stl scale=1.0 1.0 1.0
- link link_l_leg_b: geometry collision mesh filename=collision_LowerLegB.stl scale=1.0 1.0 1.0; visual mesh filename=LowerLegB.stl scale=1.0 1.0 1.0
- link link_l_leg_c: geometry collision mesh filename=collision_LowerLegC.stl scale=1.0 1.0 1.0; visual mesh filename=LowerLegC.stl scale=1.0 1.0 1.0
- link link_l_leg_d: geometry collision mesh filename=collision_LowerLegD.stl scale=1.0 1.0 1.0; visual mesh filename=LowerLegD.stl scale=1.0 1.0 1.0
Joints:
- joint link_hip_a: limit lower=-1.31 upper=2.443 effort=2.7 velocity=50.0 -> lower=-1.31 upper=2.443 effort=55 velocity=28.6
- joint link_hip_b: limit lower=-1.31 upper=2.443 effort=2.7 velocity=50.0 -> lower=-1.31 upper=2.443 effort=55 velocity=28.6
- joint link_hip_c: limit lower=-1.31 upper=2.443 effort=2.7 velocity=50.0 -> lower=-1.31 upper=2.443 effort=55 velocity=28.6
- joint link_hip_d: limit lower=-1.31 upper=2.443 effort=2.7 velocity=50.0 -> lower=-1.31 upper=2.443 effort=55 velocity=28.6
- joint link_l_leg_a: limit lower=-6.3 upper=6.3 effort=2.7 velocity=50.0 -> lower=-6.3 upper=6.3 effort=55 velocity=28.6
- joint link_l_leg_b: limit lower=-6.3 upper=6.3 effort=2.7 velocity=50.0 -> lower=-6.3 upper=6.3 effort=55 velocity=28.6
- joint link_l_leg_c: limit lower=-6.3 upper=6.3 effort=2.7 velocity=50.0 -> lower=-6.3 upper=6.3 effort=55 velocity=28.6
- joint link_l_leg_d: limit lower=-6.3 upper=6.3 effort=2.7 velocity=50.0 -> lower=-6.3 upper=6.3 effort=55 velocity=28.6
- joint link_u_leg_a: limit lower=-6.3 upper=6.3 effort=2.7 velocity=50.0 -> lower=-6.3 upper=6.3 effort=55 velocity=28.6
- joint link_u_leg_b: limit lower=-6.3 upper=6.3 effort=2.7 velocity=50.0 -> lower=-6.3 upper=6.3 effort=55 velocity=28.6
- joint link_u_leg_c: limit lower=-6.3 upper=6.3 effort=2.7 velocity=50.0 -> lower=-6.3 upper=6.3 effort=55 velocity=28.6
- joint link_u_leg_d: limit lower=-6.3 upper=6.3 effort=2.7 velocity=50.0 -> lower=-6.3 upper=6.3 effort=55 velocity=28.6

Commit message: Fix urdf issues

File: quadruped_envs/urdf/od.urdf (robot description, URDF)
Before this commit: robot od, 14 links, 13 joints
Links:
- link link_hip_a: geometry collision mesh filename=collision_HipA.stl scale=1.0 0.9 1.0; visual mesh filename=HipFeModuleA.stl scale=1.0 1.0 1.0
- link link_hip_b: geometry collision mesh filename=collision_HipB.stl scale=1.0 0.9 1.0; visual mesh filename=HipAdapterB.stl scale=1.0 1.0 1.0
- link link_hip_c: geometry collision mesh filename=collision_HipC.stl scale=1.0 1.0 1.0; visual mesh filename=HipAdapterC.stl scale=1.0 1.0 1.0
- link link_hip_d: geometry collision mesh filename=collision_HipD.stl scale=1.0 1.0 1.0; visual mesh filename=HipFeModuleD.stl scale=1.0 1.0 1.0
- link link_root: geometry collision mesh filename=collision_root.stl scale=1.0 1.0 1.0; visual mesh filename=Body_Structure.stl scale=1.0 1.0 1.0
- link link_u_leg_a: geometry collision mesh filename=collision_UpperLegA.stl scale=0.9 0.9 0.9; visual mesh filename=UpperLegModuleA.stl scale=1.0 1.0 1.0
- link link_u_leg_b: geometry collision mesh filename=collision_UpperLegB.stl scale=1.0 1.0 1.0; visual mesh filename=UpperLegModuleB.stl scale=1.0 1.0 1.0
- link link_u_leg_c: geometry collision mesh filename=collision_UpperLegC.stl scale=1.0 1.0 1.0; visual mesh filename=UpperLegModuleC.stl scale=1.0 1.0 1.0
- link link_u_leg_d: geometry collision mesh filename=collision_UpperLegD.stl scale=1.0 1.0 1.0; visual mesh filename=UpperLegModuleD.stl scale=1.0 1.0 1.0

Commit message: Fixed robot urdf

File: quadruped_envs/urdf/od.urdf (robot description, URDF)
Before this commit: robot od, 14 links, 13 joints
Links:
- link link_hip_a: geometry collision mesh filename=collision_HipA.stl scale=1.0 1.0 1.0; visual mesh filename=HipFeModuleA.stl scale=1.0 1.0 1.0
- link link_hip_b: geometry collision mesh filename=collision_HipB.stl scale=1.0 1.0 1.0; visual mesh filename=HipAdapterB.stl scale=1.0 1.0 1.0
- link link_u_leg_a: geometry collision mesh filename=collision_UpperLegA.stl scale=1.0 1.0 1.0; visual mesh filename=UpperLegModuleA.stl scale=1.0 1.0 1.0
Joints:
- joint link_l_leg_a: origin xyz=0.10112 -0.05695 -0.12354 rpy=0 0 0 -> xyz=0.1004 -0.05695 -0.124 rpy=0 0 0
- joint link_l_leg_b: origin xyz=0.10112 0.05695 -0.12354 rpy=0 0 0 -> xyz=0.1004 0.05695 -0.124 rpy=0 0 0
- joint link_l_leg_c: origin xyz=0.09841 -0.05695 -0.12588 rpy=0 0 0 -> xyz=0.09902 -0.05695 -0.12527 rpy=0 0 0
- joint link_l_leg_d: origin xyz=0.09841 0.05695 -0.12588 rpy=0 -1.34948 0 -> xyz=0.09902 0.05695 -0.12527 rpy=0 0 0

Commit message: Fixed robot mass

File: quadruped_envs/urdf/od.urdf (robot description, URDF)
Before this commit: robot od, 14 links, 13 joints
Links:
- link imu_link: mass 0.001 -> 0.01
- link link_hip_a: mass 0.15 -> 1.5
- link link_hip_b: mass 0.15 -> 1.5
- link link_hip_c: mass 0.15 -> 1.5
- link link_hip_d: mass 0.15 -> 1.5
- link link_l_leg_a: mass 0.02 -> 0.2
- link link_l_leg_b: mass 0.02 -> 0.2
- link link_l_leg_c: mass 0.02 -> 0.2
- link link_l_leg_d: mass 0.02 -> 0.2
- link link_u_leg_a: mass 0.15 -> 1.5
- link link_u_leg_b: mass 0.15 -> 1.5
- link link_u_leg_c: mass 0.15 -> 1.5
- link link_u_leg_d: mass 0.15 -> 1.5

Commit message: Add motion retargeting script

File: quadruped_envs/urdf/od.urdf (robot description, URDF)
Before this commit: robot od, 14 links, 13 joints
Joints:
- joint link_hip_a: axis -1.0 0 0 -> 1.0 0 0; limit lower=-1.31 upper=2.443 effort=55 velocity=28.6 -> lower=-1.31 upper=2.443 effort=2.7 velocity=50.0; origin xyz=-0.1939 -0.09 0 rpy=0 0 0 -> xyz=0.1939 0.09 0 rpy=0 0 0
- joint link_hip_b: axis -1.0 0 0 -> 1.0 0 0; limit lower=-1.31 upper=2.443 effort=55 velocity=28.6 -> lower=-1.31 upper=2.443 effort=2.7 velocity=50.0; origin xyz=-0.1939 0.09 0 rpy=0 0 0 -> xyz=0.1939 -0.09 0 rpy=0 0 0
- joint link_hip_c: limit lower=-1.31 upper=2.443 effort=55 velocity=28.6 -> lower=-1.31 upper=2.443 effort=2.7 velocity=50.0; origin xyz=0.1939 -0.09 0 rpy=0 0 0 -> xyz=-0.1939 0.09 0 rpy=0 0 0
- joint link_hip_d: limit lower=-1.31 upper=2.443 effort=55 velocity=28.6 -> lower=-1.31 upper=2.443 effort=2.7 velocity=50.0; origin xyz=0.1939 0.09 0 rpy=0 0 0 -> xyz=-0.1939 -0.09 0 rpy=0 0 0
- joint link_l_leg_a: axis 0 -1.0 0 -> 0 1.0 0; limit lower=-6.3 upper=6.3 effort=55 velocity=28.6 -> lower=-6.3 upper=6.3 effort=2.7 velocity=50.0; origin xyz=0.1004 -0.05695 -0.124 rpy=0 0 0 -> xyz=-0.1004 0.05695 -0.124 rpy=0 0 0
- joint link_l_leg_b: limit lower=-6.3 upper=6.3 effort=55 velocity=28.6 -> lower=-6.3 upper=6.3 effort=2.7 velocity=50.0; origin xyz=0.1004 0.05695 -0.124 rpy=0 0 0 -> xyz=-0.1004 -0.05695 -0.124 rpy=0 0 0
- joint link_l_leg_c: axis 0 -1.0 0 -> 0 1.0 0; limit lower=-6.3 upper=6.3 effort=55 velocity=28.6 -> lower=-6.3 upper=6.3 effort=2.7 velocity=50.0; origin xyz=0.09902 -0.05695 -0.12527 rpy=0 0 0 -> xyz=-0.09902 0.05695 -0.12527 rpy=0 0 0
- joint link_l_leg_d: limit lower=-6.3 upper=6.3 effort=55 velocity=28.6 -> lower=-6.3 upper=6.3 effort=2.7 velocity=50.0; origin xyz=0.09902 0.05695 -0.12527 rpy=0 0 0 -> xyz=-0.09902 -0.05695 -0.12527 rpy=0 0 0
- joint link_u_leg_a: axis 0 -1.0 0 -> 0 1.0 0; limit lower=-6.3 upper=6.3 effort=55 velocity=28.6 -> lower=-6.3 upper=6.3 effort=2.7 velocity=50.0
- joint link_u_leg_b: limit lower=-6.3 upper=6.3 effort=55 velocity=28.6 -> lower=-6.3 upper=6.3 effort=2.7 velocity=50.0
- joint link_u_leg_c: axis 0 -1.0 0 -> 0 1.0 0; limit lower=-6.3 upper=6.3 effort=55 velocity=28.6 -> lower=-6.3 upper=6.3 effort=2.7 velocity=50.0
- joint link_u_leg_d: limit lower=-6.3 upper=6.3 effort=55 velocity=28.6 -> lower=-6.3 upper=6.3 effort=2.7 velocity=50.0
